Commit message: Hm

File: crx_description/urdf/crx10ia_l/crx10ia_l.urdf (robot description, URDF)
Before this commit: robot crx10ia_l, 13 links, 12 joints
Links:
- removed link flange1
- removed link tcp
- removed link tcp_left
- removed link tcp_right
Joints:
- removed joint flange-flange1
- removed joint flange1-tcp
- removed joint tcp-tcp_left
- removed joint tcp-tcp_right
